File: led_ring.kicad_sch (KiCad schematic)
At the start: 25 parts

Commit message: Change LEDs in bom
Parts:
- D1, D10, D11, D12, D2, D3, D4, D5, D6, D7, D8, D9: Supplier https://www.digikey.ch/en/products/detail/adafruit-industri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 -> https://www.digikey.ch/en/products/detail/inolux/IN-PI15TAT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
Changed lines of the file:
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@@
 			)
 		)
-		(property "Datasheet" "https://mm.digikey.com/Volume0/opasdata/d220001/medias/docus/2384/CL05A105KP5NNN_Specsheet%20(1).pdf"
+		(property "Datasheet" "https://www.inolux-corp.com/datasheet/SMDLED/Addressable%20LED/IN-PI15TAT5R5G5B_v1.0.pdf"
 			(at 250.19 61.595 0)
 			(effects
@@
 			)
 		)
-		(property "Supplier" "https://www.digikey.ch/en/products/detail/adafruit-industries-llc/4492/11569136"
+		(property "Supplier" "https://www.digikey.ch/en/products/detail/inolux/IN-PI15TAT5R5G5B/14555725"
 			(at 247.65 52.07 0)
 			(effects
@@
 			)
 		)
-		(property "Datasheet" "https://mm.digikey.com/Volume0/opasdata/d220001/medias/docus/2384/CL05A105KP5NNN_Specsheet%20(1).pdf"
+		(property "Datasheet" "https://www.inolux-corp.com/datasheet/SMDLED/Addressable%20LED/IN-PI15TAT5R5G5B_v1.0.pdf"
 			(at 125.73 61.595 0)
 			(effects
@@
 			)
 		)
-		(property "Supplier" "https://www.digikey.ch/en/products/detail/adafruit-industries-llc/4492/11569136"
+		(property "Supplier" "https://www.digikey.ch/en/products/detail/inolux/IN-PI15TAT5R5G5B/14555725"
 			(at 123.19 52.07 0)
 			(effects
@@
 			)
 		)
-		(property "Datasheet" "https://mm.digikey.com/Volume0/opasdata/d220001/medias/docus/2384/CL05A105KP5NNN_Specsheet%20(1).pdf"
+		(property "Datasheet" "https://www.inolux-corp.com/datasheet/SMDLED/Addressable%20LED/IN-PI15TAT5R5G5B_v1.0.pdf"
 			(at 72.39 61.595 0)
 			(effects
@@
 			)
 		)
-		(property "Supplier" "https://www.digikey.ch/en/products/detail/adafruit-industries-llc/4492/11569136"
+		(property "Supplier" "https://www.digikey.ch/en/products/detail/inolux/IN-PI15TAT5R5G5B/14555725"
 			(at 69.85 52.07 0)
 			(effects
@@
 			)
 		)
-		(property "Datasheet" "https://mm.digikey.com/Volume0/opasdata/d220001/medias/docus/2384/CL05A105KP5NNN_Specsheet%20(1).pdf"
+		(property "Datasheet" "https://www.inolux-corp.com/datasheet/SMDLED/Addressable%20LED/IN-PI15TAT5R5G5B_v1.0.pdf"
 			(at 143.51 61.595 0)
 			(effects
@@
 			)
 		)
-		(property "Supplier" "https://www.digikey.ch/en/products/detail/adafruit-industries-llc/4492/11569136"
+		(property "Supplier" "https://www.digikey.ch/en/products/detail/inolux/IN-PI15TAT5R5G5B/14555725"
 			(at 140.97 52.07 0)
 			(effects
@@
 			)
 		)
-		(property "Datasheet" "https://mm.digikey.com/Volume0/opasdata/d220001/medias/docus/2384/CL05A105KP5NNN_Specsheet%20(1).pdf"
+		(property "Datasheet" "https://www.inolux-corp.com/datasheet/SMDLED/Addressable%20LED/IN-PI15TAT5R5G5B_v1.0.pdf"
 			(at 179.07 61.595 0)
 			(effects
@@
 			)
 		)
-		(property "Supplier" "https://www.digikey.ch/en/products/detail/adafruit-industries-llc/4492/11569136"
+		(property "Supplier" "https://www.digikey.ch/en/products/detail/inolux/IN-PI15TAT5R5G5B/14555725"
 			(at 176.53 52.07 0)
 			(effects
@@
 			)
 		)
-		(property "Datasheet" "https://mm.digikey.com/Volume0/opasdata/d220001/medias/docus/2384/CL05A105KP5NNN_Specsheet%20(1).pdf"
+		(property "Datasheet" "https://www.inolux-corp.com/datasheet/SMDLED/Addressable%20LED/IN-PI15TAT5R5G5B_v1.0.pdf"
 			(at 232.41 61.595 0)
 			(effects
@@
 			)
 		)
-		(property "Supplier" "https://www.digikey.ch/en/products/detail/adafruit-industries-llc/4492/11569136"
+		(property "Supplier" "https://www.digikey.ch/en/products/detail/inolux/IN-PI15TAT5R5G5B/14555725"
 			(at 229.87 52.07 0)
 			(effects
@@
 			)
 		)
-		(property "Datasheet" "https://mm.digikey.com/Volume0/opasdata/d220001/medias/docus/2384/CL05A105KP5NNN_Specsheet%20(1).pdf"
+		(property "Datasheet" "https://www.inolux-corp.com/datasheet/SMDLED/Addressable%20LED/IN-PI15TAT5R5G5B_v1.0.pdf"
 			(at 107.95 61.595 0)
 			(effects
@@
 			)
 		)
-		(property "Supplier" "https://www.digikey.ch/en/products/detail/adafruit-industries-llc/4492/11569136"
+		(property "Supplier" "https://www.digikey.ch/en/products/detail/inolux/IN-PI15TAT5R5G5B/14555725"
 			(at 105.41 52.07 0)
 			(effects
@@
 			)
 		)
-		(property "Datasheet" "https://mm.digikey.com/Volume0/opasdata/d220001/medias/docus/2384/CL05A105KP5NNN_Specsheet%20(1).pdf"
+		(property "Datasheet" "https://www.inolux-corp.com/datasheet/SMDLED/Addressable%20LED/IN-PI15TAT5R5G5B_v1.0.pdf"
 			(at 161.29 61.595 0)
 			(effects
@@
 			)
 		)
-		(property "Supplier" "https://www.digikey.ch/en/products/detail/adafruit-industries-llc/4492/11569136"
+		(property "Supplier" "https://www.digikey.ch/en/products/detail/inolux/IN-PI15TAT5R5G5B/14555725"
 			(at 158.75 52.07 0)
 			(effects
@@
 			)
 		)
-		(property "Datasheet" "https://mm.digikey.com/Volume0/opasdata/d220001/medias/docus/2384/CL05A105KP5NNN_Specsheet%20(1).pdf"
+		(property "Datasheet" "https://www.inolux-corp.com/datasheet/SMDLED/Addressable%20LED/IN-PI15TAT5R5G5B_v1.0.pdf"
 			(at 90.17 61.595 0)
 			(effects
@@
 			)
 		)
-		(property "Supplier" "https://www.digikey.ch/en/products/detail/adafruit-industries-llc/4492/11569136"
+		(property "Supplier" "https://www.digikey.ch/en/products/detail/inolux/IN-PI15TAT5R5G5B/14555725"
 			(at 87.63 52.07 0)
 			(effects
@@
 			)
 		)
-		(property "Datasheet" "https://mm.digikey.com/Volume0/opasdata/d220001/medias/docus/2384/CL05A105KP5NNN_Specsheet%20(1).pdf"
+		(property "Datasheet" "https://www.inolux-corp.com/datasheet/SMDLED/Addressable%20LED/IN-PI15TAT5R5G5B_v1.0.pdf"
 			(at 54.61 61.595 0)
 			(effects
@@
 			)
 		)
-		(property "Supplier" "https://www.digikey.ch/en/products/detail/adafruit-industries-llc/4492/11569136"
+		(property "Supplier" "https://www.digikey.ch/en/products/detail/inolux/IN-PI15TAT5R5G5B/14555725"
 			(at 52.07 52.07 0)
 			(effects
@@
 			)
 		)
-		(property "Datasheet" "https://mm.digikey.com/Volume0/opasdata/d220001/medias/docus/2384/CL05A105KP5NNN_Specsheet%20(1).pdf"
+		(property "Datasheet" "https://www.inolux-corp.com/datasheet/SMDLED/Addressable%20LED/IN-PI15TAT5R5G5B_v1.0.pdf"
 			(at 196.85 61.595 0)
 			(effects
@@
 			)
 		)
-		(property "Supplier" "https://www.digikey.ch/en/products/detail/adafruit-industries-llc/4492/11569136"
+		(property "Supplier" "https://www.digikey.ch/en/products/detail/inolux/IN-PI15TAT5R5G5B/14555725"
 			(at 194.31 52.07 0)
 			(effects
@@
 			)
 		)
-		(property "Datasheet" "https://mm.digikey.com/Volume0/opasdata/d220001/medias/docus/2384/CL05A105KP5NNN_Specsheet%20(1).pdf"
+		(property "Datasheet" "https://www.inolux-corp.com/datasheet/SMDLED/Addressable%20LED/IN-PI15TAT5R5G5B_v1.0.pdf"
 			(at 214.63 61.595 0)
 			(effects
@@
 			)
 		)
-		(property "Supplier" "https://www.digikey.ch/en/products/detail/adafruit-industries-llc/4492/11569136"
+		(property "Supplier" "https://www.digikey.ch/en/products/detail/inolux/IN-PI15TAT5R5G5B/14555725"
 			(at 212.09 52.07 0)
 			(effects
