File: pedalboard-display.kicad_sch (KiCad schematic)
At the start: 22 parts, among them J1 LED-IN, J2 LED-OUT, J3 OLED

Commit message: Improve BOM
Parts:
- J1: value LED-IN -> JST PH 3
- J2: value LED-OUT -> JST PH 3
- J3: value OLED -> JST PH 4
- R2, R3: Supplier (none) -> https://www.digikey.ch/en/products/detail/stackpole-electro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
- U1, U2: value ~ -> OLED I2C; Supplier (none) -> https://www.aliexpress.com/item/1005005253671396.html
Changed lines of the file:
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@@
 			)
 		)
-		(property "Value" "LED-IN"
+		(property "Value" "JST PH 3"
 			(at 145.415 35.56 0)
 			(effects
@@
 			)
 		)
-		(property "Value" "~"
+		(property "Value" "OLED I2C"
 			(at 130.81 176.53 0)
 			(effects
@@
 			)
 		)
-		(property "Datasheet" ""
+		(property "Datasheet" "img/GME12812.pdf"
 			(at 119.38 176.53 0)
 			(effects
@@
 		)
 		(property "Description" ""
+			(at 119.38 176.53 0)
+			(effects
+				(font
+					(size 1.27 1.27)
+				)
+				(hide yes)
+			)
+		)
+		(property "Supplier" "https://www.aliexpress.com/item/1005005253671396.html"
 			(at 119.38 176.53 0)
 			(effects
@@
 			)
 		)
-		(property "Datasheet" "~"
+		(property "Datasheet" "https://www.seielect.com/catalog/sei-rmcf_rmcp.pdf"
 			(at 83.82 172.72 0)
 			(effects
@@
 		)
 		(property "Description" "Resistor"
+			(at 83.82 172.72 0)
+			(effects
+				(font
+					(size 1.27 1.27)
+				)
+				(hide yes)
+			)
+		)
+		(property "Supplier" "https://www.digikey.ch/en/products/detail/stackpole-electronics-inc/RMCF0805FT3K30/1760325"
 			(at 83.82 172.72 0)
 			(effects
@@
 			)
 		)
-		(property "Datasheet" "~"
+		(property "Datasheet" "https://www.seielect.com/catalog/sei-rmcf_rmcp.pdf"
 			(at 83.82 170.18 0)
 			(effects
@@
 		)
 		(property "Description" "Resistor"
+			(at 83.82 170.18 0)
+			(effects
+				(font
+					(size 1.27 1.27)
+				)
+				(hide yes)
+			)
+		)
+		(property "Supplier" "https://www.digikey.ch/en/products/detail/stackpole-electronics-inc/RMCF0805FT3K30/1760325"
 			(at 83.82 170.18 0)
 			(effects
@@
 			)
 		)
-		(property "Value" "LED-OUT"
+		(property "Value" "JST PH 3"
 			(at 114.935 133.35 0)
 			(effects
@@
 			)
 		)
-		(property "Value" "~"
+		(property "Value" "OLED I2C"
 			(at 171.45 176.53 0)
 			(effects
@@
 			)
 		)
-		(property "Datasheet" ""
+		(property "Datasheet" "img/GME12812.pdf"
 			(at 160.02 176.53 0)
 			(effects
@@
 			)
 		)
+		(property "Supplier" "https://www.aliexpress.com/item/1005005253671396.html"
+			(at 160.02 176.53 0)
+			(effects
+				(font
+					(size 1.27 1.27)
+				)
+				(hide yes)
+			)
+		)
 		(pin "4"
 		)
@@
 			)
 		)
-		(property "Value" "OLED"
+		(property "Value" "JST PH 4"
 			(at 67.945 167.64 0)
 			(effects

Commit message: Change LEDs in bom
Parts:
- D97, D98: Supplier https://www.digikey.ch/en/products/detail/adafruit-industri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 -> https://www.digikey.ch/en/products/detail/inolux/IN-PI15TAT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
Changed lines of the file:
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@@
 			)
 		)
-		(property "Datasheet" "https://mm.digikey.com/Volume0/opasdata/d220001/medias/docus/2384/CL05A105KP5NNN_Specsheet%20(1).pdf"
+		(property "Datasheet" "https://www.inolux-corp.com/datasheet/SMDLED/Addressable%20LED/IN-PI15TAT5R5G5B_v1.0.pdf"
 			(at 67.31 135.255 0)
 			(effects
@@
 			)
 		)
-		(property "Supplier" "https://www.digikey.ch/en/products/detail/adafruit-industries-llc/4492/11569136"
+		(property "Supplier" "https://www.digikey.ch/en/products/detail/inolux/IN-PI15TAT5R5G5B/14555725"
 			(at 64.77 125.73 0)
 			(effects
@@
 			)
 		)
-		(property "Datasheet" "https://mm.digikey.com/Volume0/opasdata/d220001/medias/docus/2384/CL05A105KP5NNN_Specsheet%20(1).pdf"
+		(property "Datasheet" "https://www.inolux-corp.com/datasheet/SMDLED/Addressable%20LED/IN-PI15TAT5R5G5B_v1.0.pdf"
 			(at 93.98 135.255 0)
 			(effects
@@
 			)
 		)
-		(property "Supplier" "https://www.digikey.ch/en/products/detail/adafruit-industries-llc/4492/11569136"
+		(property "Supplier" "https://www.digikey.ch/en/products/detail/inolux/IN-PI15TAT5R5G5B/14555725"
 			(at 91.44 125.73 0)
 			(effects

Commit message: Improve BOM (JST)
Parts:
- J1, J2, J3: Supplier (none) -> https://www.digikey.ch/de/products/detail/jst-sales-america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
Changed lines of the file:
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@@
 			)
 		)
-		(property "Datasheet" "~"
+		(property "Datasheet" "https://www.jst-mfg.com/product/pdf/eng/ePH.pdf"
 			(at 144.78 40.64 0)
 			(effects
@@
 		)
 		(property "Description" ""
+			(at 144.78 40.64 0)
+			(effects
+				(font
+					(size 1.27 1.27)
+				)
+				(hide yes)
+			)
+		)
+		(property "Supplier" "https://www.digikey.ch/de/products/detail/jst-sales-america-inc/B3B-PH-SM4-TB/926832"
 			(at 144.78 40.64 0)
 			(effects
@@
 			)
 		)
-		(property "Datasheet" "~"
+		(property "Datasheet" "https://www.jst-mfg.com/product/pdf/eng/ePH.pdf"
 			(at 115.57 128.27 0)
 			(effects
@@
 		)
 		(property "Description" ""
+			(at 115.57 128.27 0)
+			(effects
+				(font
+					(size 1.27 1.27)
+				)
+				(hide yes)
+			)
+		)
+		(property "Supplier" "https://www.digikey.ch/de/products/detail/jst-sales-america-inc/B3B-PH-SM4-TB/926832"
 			(at 115.57 128.27 0)
 			(effects
@@
 			)
 		)
-		(property "Datasheet" "~"
+		(property "Datasheet" "https://www.jst-mfg.com/product/pdf/eng/ePH.pdf"
 			(at 67.31 172.72 0)
 			(effects
@@
 			(at 67.31 172.72 0)
 			(effects
+				(font
+					(size 1.27 1.27)
+				)
+				(hide yes)
+			)
+		)
+		(property "Supplier" "https://www.digikey.ch/de/products/detail/jst-sales-america-inc./B4B-PH-SM4-TB/926833"
+			(at 67.31 172.72 0)
+			(effects

Commit message: Add I2C addresses of the displays
Other:
- note added: "Display Left: I2C address: 0x3C (original)"
- note added: "Display Left: I2C address: 0x3D (modified)"
Changed lines of the file:
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@@
 		)
 	)
-	(label "I2C_SDA"
-		(at 106.68 170.18 180)
-		(fields_autoplaced yes)
+	(text "Display Left:\nI2C address: 0x3C (original)"
+		(exclude_from_sim no)
+		(at 160.274 156.464 0)
 		(effects
 			(font
 				(size 1.27 1.27)
 			)
-			(justify right bottom)
-		)
-	)
-	(label "I2C_SCL"
-		(at 147.32 167.64 180)
-		(fields_autoplaced yes)
+		)
+	)
+	(text "Display Left:\nI2C address: 0x3D (modified)"
+		(exclude_from_sim no)
+		(at 119.634 156.464 0)
 		(effects
 			(font
 				(size 1.27 1.27)
 			)
-			(justify right bottom)
 		)
 	)
 	(label "I2C_SDA"
-		(at 147.32 170.18 180)
+		(at 106.68 170.18 180)
 		(fields_autoplaced yes)
 		(effects
@@
 	)
 	(label "I2C_SCL"
-		(at 106.68 167.64 180)
+		(at 147.32 167.64 180)
 		(fields_autoplaced yes)
 		(effects
@@
 	)
 	(label "I2C_SDA"
-		(at 72.39 172.72 0)
+		(at 147.32 170.18 180)
 		(fields_autoplaced yes)
 		(effects
@@
 				(size 1.27 1.27)
 			)
-			(justify left bottom)
+			(justify right bottom)
 		)
 	)
 	(label "I2C_SCL"
-		(at 72.39 170.18 0)
+		(at 106.68 167.64 180)
 		(fields_autoplaced yes)
 		(effects
@@
 				(size 1.27 1.27)
 			)
+			(justify right bottom)
+		)
+	)
+	(label "I2C_SDA"
+		(at 72.39 172.72 0)
+		(fields_autoplaced yes)
+		(effects
+			(font
+				(size 1.27 1.27)
+			)
+			(justify left bottom)
+		)
+	)
+	(label "I2C_SCL"
+		(at 72.39 170.18 0)
+		(fields_autoplaced yes)
+		(effects
+			(font
+				(size 1.27 1.27)
+			)
 			(justify left bottom)
 		)
@@
 		(on_board yes)
 		(dnp no)
-		(fields_autoplaced yes)
 		(property "Reference" "#PWR042"
 			(at 160.02 166.37 0)
@@
 		)
 		(property "Value" "+3.3V"
-			(at 160.02 157.48 0)
+			(at 164.592 162.56 0)
 			(effects
 				(font
@@
 		(on_board yes)
 		(dnp no)
-		(fields_autoplaced yes)
 		(property "Reference" "#PWR041"
 			(at 119.38 166.37 0)
@@
 		)
 		(property "Value" "+3.3V"
-			(at 119.38 157.48 0)
-			(effects
-				(font
+			(at 123.19 162.56 0)
+			(effects
+				(font

Commit message: Fix text
Other:
- note added: "Display Right: I2C address: 0x3C (original)"
- note removed: "Display Left: I2C address: 0x3C (original)"
Changed lines of the file:
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@@
 		)
 	)
-	(text "Display Left:\nI2C address: 0x3C (original)"
+	(text "Display Right:\nI2C address: 0x3C (original)"
 		(exclude_from_sim no)
 		(at 160.274 156.464 0)
@@
 		(on_board yes)
 		(dnp no)
-		(fields_autoplaced yes)
 		(property "Reference" "U1"
-			(at 130.81 174.6249 0)
+			(at 123.952 187.8329 0)
 			(effects
 				(font
@@
 		)
 		(property "Value" "OLED I2C"
-			(at 130.81 176.53 0)
+			(at 123.952 189.738 0)
 			(effects
 				(font
@@
 		(on_board yes)
 		(dnp no)
-		(fields_autoplaced yes)
 		(property "Reference" "U2"
-			(at 171.45 174.6249 0)
+			(at 165.862 188.214 0)
 			(effects
 				(font
@@
 		)
 		(property "Value" "OLED I2C"
-			(at 171.45 176.53 0)
-			(effects
-				(font
+			(at 165.862 190.246 0)
+			(effects
+				(font
